File: millipad/millipad.kicad_pcb (KiCad board)
At the start: 2 copper layers, 131.8 x 76.2 mm, 58 parts, among them J1 6P6C, SW1 SW_Push, SW2 Rotary_Encoder_Switch, SW3 SW_Push, SW4 SW_Push, U1 ATmega32U4-AU, U2 PRTR5V0U2X, Y1 16MHz

Commit message: ground planes
Routing:
- added copper zone on F.Cu, net KEYBOARD_GND
